Commit message: 4/14 rviz with drone urdf running

File: urdf/quad.urdf.xacro (robot description, xacro)
@@ -13,5 +13,5 @@
       <origin rpy="0 0 0" xyz="0 0 0"/>
       <geometry>
-        <mesh filename="quadrotor_base.obj" scale=".1 .1 .1"/>
+        <mesh filename="package://my_package/meshes/quadrotor_base.obj" scale="0.1 0.1 0.1"/>
       </geometry>
     </visual>

Commit message: added rviz config, urdf tf, added config to cmake

File: urdf/quad.urdf.xacro (robot description, xacro)
@@ -4,4 +4,10 @@
  xmlns:xsi="http://www.w3.org/2001/XMLSchema-instance"
  xsi:schemaLocation="http://drake.mit.edu ../../../../pods/drake/doc/drakeURDF.xsd" name="quadrotor">
+  <link name="world_link"/>
+  <joint name="world_to_base" type="fixed">
+    <parent link="world_link"/>
+    <child  link="base_link"/>
+    <origin xyz="0 0 0" rpy="0 0 0"/>
+  </joint>
   <link name="base_link">
     <inertial>

Commit message: 4/24 changed lauch file with dummy world link

File: urdf/quad.urdf.xacro (robot description, xacro)
@@ -4,10 +4,10 @@
  xmlns:xsi="http://www.w3.org/2001/XMLSchema-instance"
  xsi:schemaLocation="http://drake.mit.edu ../../../../pods/drake/doc/drakeURDF.xsd" name="quadrotor">
-  <link name="world_link"/>
+  <!--<link name="world_link"/>
   <joint name="world_to_base" type="fixed">
     <parent link="world_link"/>
     <child  link="base_link"/>
     <origin xyz="0 0 0" rpy="0 0 0"/>
-  </joint>
+  </joint>-->
   <link name="base_link">
     <inertial>
